File: Eagle/monitor_12.sch (EAGLE design)
At the start: 43 parts, among them IC1 74HC574N, IC2 74HC04N, IC3 74HC574N, IC5 74HC574N, IC6 74HC574N

Commit message: Added files via upload
Other:
- note added: "Address Bus or Program Counter"
- note removed: "Adress Bus or Program Counter"
Changed lines of the file:
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@@
 <text x="175.26" y="71.12" size="1.778" layer="91">Low</text>
 <text x="175.26" y="33.02" size="1.778" layer="91">High</text>
-<text x="45.72" y="175.26" size="6.4516" layer="91">Adress Bus or Program Counter</text>
+<text x="45.72" y="175.26" size="6.4516" layer="91">Address Bus or Program Counter</text>
 </plain>
 <instances>
